File: hw/sch_pcb/DATALOGGER02A.kicad_sch (KiCad schematic)
At the start: 68 parts

Commit message: IMU schema
Parts:
- added C?: 47uF, Mlab_C:TantalC_SizeC_Reflow, symbol DATALOGGER01A-rescue:CP-device
- added C? (x5): 100nF, Mlab_R:SMD-0603, symbol Device:C
- added C?: 100nF, Mlab_R:SMD-0805, symbol DATALOGGER01A-rescue:C-device
- added C?: EMI_Filter_C, Mlab_L:FIR1, symbol DATALOGGER01A-rescue:EMI_Filter_C-device
- added C? (x2): 1uF, Mlab_R:SMD-0603, symbol Device:C
- added D?: M4, Mlab_D:SMA_Standard, symbol DATALOGGER01A-rescue:D-device
- added F?: 750mA, Mlab_F:1812, symbol DATALOGGER01A-rescue:Polyfuse-device
- added J? (x8): HEADER_2x01_PARALLEL, Mlab_Pin_Headers:Straight_2x01, symbol DATALOGGER01A-rescue:HEADER_2x01_PARALLEL-MLAB_HEADER
- added R? (x4): 10k, Mlab_R:SMD-0603, symbol Device:R
- added R?: 0R, Mlab_R:SMD-0603, symbol Device:R
- added R?: -, Mlab_R:SMD-0603, symbol Device:R
- added R? (x2): 10k, Mlab_R:SMD-0805, symbol DATALOGGER01A-rescue:R-device
- added SW?: 5MS1S102AM6QE, Mlab_SW:5MS1S102AM6QE, symbol Switch:SW_SPST
- added U?: TXS0108EPW, Package_SO:TSSOP-20_4.4x6.5mm_P0.65mm, symbol Logic_LevelTranslator:TXS0108EPW
- added U?: ICM-20948, Sensor_Motion:InvenSense_QFN-24_3x3mm_P0.4mm, symbol Sensor_Motion:ICM-20948
- added U?: MIC5504-1.8YM5-TR, Package_TO_SOT_SMD:SOT-23-5, symbol Regulator_Linear:MIC5504-1.8YM5
Connections:
- net GND: now also C?.1, C?.2, C?.2, C?.2, C?.2, C?.2, C?.2, C?.2, C?.2, C?.2, D?.2 (A), J?.1, J?.1, J?.1, J?.1, J?.2, J?.2, J?.2, J?.2, R?.2, U?.11 (FSYNC), U?.11 (GND), U?.18 (GND), U?.2 (GND), U?.20 (GND)
- net PB0: now also U?.16 (B4)
- net PB5: now also U?.14 (B6)
- net PB6: now also U?.18 (B2)
- net PB7: now also U?.13 (B7)
- net VDD: now also C?.1, C?.3
- new net: D?.1 (K), F?.1
- new net: F?.2, J?.1, J?.2
- new net: C?.1, C?.1
- new net: C?.1, U?.10 (REGOUT)
- new net !CS_1V8: U?.22 (~{CS}), U?.5 (A4)
- new net +1V8: C?.1, C?.1, C?.2, R?.1, R?.1, R?.1, R?.1, R?.1, U?.10 (OE), U?.2 (VCCA), U?.5 (VOUT), U?.8 (VDDIO)
- new net +3.3V: C?.1, J?.1, J?.2, R?.2, R?.2, U?.1 (VIN), U?.3 (EN)
- new net +3V3: C?.1, C?.1, U?.13 (VDD), U?.19 (VCCB)
- new net AUX_SCL_1V8: R?.2, U?.4 (A3), U?.7 (AUX_CL)
- new net AUX_SCL_3V3: J?.1, J?.2, R?.1, U?.17 (B3)
- new net AUX_SDA_1V8: R?.2, U?.21 (AUX_DA), U?.6 (A5)
- new net AUX_SDA_3V3: J?.1, J?.2, R?.1, U?.15 (B5)
- new net INT1_1V8: U?.1 (A1), U?.12 (INT1)
- new net INT1_3V3: U?.20 (B1)
- new net MISO_1V8: R?.1, R?.2, U?.3 (A2), U?.9 (SDO/AD0)
- new net MOSI_1V8: R?.2, U?.24 (SDA/SDI), U?.7 (A6)
- new net SCK_1V8: R?.2, U?.23 (SCL/SCLK), U?.8 (A7)
- no-connect marks 5 -> 7
Other:
- removed sheet Power_supply
- note added: "ANALOG CONN"
- note added: "AUX_I2C CONN"
- note added: "INERTIAL MEASUREMENT UNIT"
- note added: "Nepochopil jsme, jestli vzpinac ano nebo ne + SPINANY ZDROJ + SUPERCAP"
- note added: "PB4 - CS SD CARD PB5 - MOSI PB6 - MISO PB7 - SCK PB2 - CS FRAM PB0 - CS IMU PB3 - CS CONNECTOR PB1 - CS CONNECTOR"
- note added: "PIXHAWK STANDARD HEADERS"
- note removed: "PB4 - CS SD CARD PB5 - MOSI PB6 - MISO PB7 - SCK PB2 - CS FRAM PB3 - CS CONNECTOR"
- note removed: "PIXHAWK STANDARD"
- moved on the sheet: J?
